Commit message: caster wheel

File: urdf/dbot_mobile.urdf.xacro (robot description, xacro)
@@ -35,5 +35,5 @@
             </geometry>
         </collision>
-        <xacro:inertial_box mass="1.0" x="${chassis_l}" y="${chassis_w}" z="${chassis_h}">
+        <xacro:inertial_box mass="0.5" x="${chassis_l}" y="${chassis_w}" z="${chassis_h}">
             <origin xyz="${chassis_l/2} 0 ${chassis_h/2}"/>
         </xacro:inertial_box>
@@ -59,5 +59,5 @@
             </geometry>
         </collision>
-        <xacro:inertial_cylinder mass="1.0" length="${wheel_l}" radius="${wheel_r}">
+        <xacro:inertial_cylinder mass="0.1" length="${wheel_l}" radius="${wheel_r}">
             <origin xyz="0 0 0" rpy="0 0 0"/>
         </xacro:inertial_cylinder>
@@ -83,7 +83,31 @@
             </geometry>
         </collision>
-        <xacro:inertial_cylinder mass="1.0" length="${wheel_l}" radius="${wheel_r}">
+        <xacro:inertial_cylinder mass="0.1" length="${wheel_l}" radius="${wheel_r}">
             <origin xyz="0 0 0" rpy="0 0 0"/>
         </xacro:inertial_cylinder>
     </link>
+    <!-- Caster Wheel Joint -->
+    <joint name="caster_wheel_joint" type="fixed">
+        <origin xyz="0.24 0.0 0.0" rpy="0.0 0.0 0.0"/>
+        <parent link="chassis_link"/>
+        <child link="caster_wheel_link"/>
+        <axis xyz="0.0 0.0 -1.0"/>
+    </joint>
+    <!-- Caster Wheel Link -->
+    <link name="caster_wheel_link">
+        <visual>
+            <geometry>
+                <sphere radius="${wheel_r}"/>
+            </geometry>
+            <material name="black"/>
+        </visual>
+        <collision>
+            <geometry>
+                <sphere radius="${wheel_r}"/>
+            </geometry>
+        </collision>
+        <xacro:inertial_sphere mass="0.1" radius="${wheel_r}">
+            <origin xyz="0 0 0" rpy="0 0 0"/>
+        </xacro:inertial_sphere>
+    </link>
 </robot>

Commit message: urdf split

File: urdf/dbot_mobile.urdf.xacro (robot description, xacro)
@@ -3,111 +3,7 @@
     <!-- Commmon data for the robot. -->
     <xacro:include filename="robot_common.xacro"/>
-    <!-- Chassis size -->
-    <xacro:property name="chassis_l" value="0.300" />
-    <xacro:property name="chassis_w" value="0.300" />
-    <xacro:property name="chassis_h" value="0.150" />
-    <!-- Wheel size -->
-    <xacro:property name="wheel_r" value="0.05" />
-    <xacro:property name="wheel_l" value="0.04" />
-    <!-- The first link of the robot -->
-    <!-- Fixed base-->
-    <link name="base_link">
-    </link>
-    <!-- Chassis Joint -->
-    <joint name="chassis_joint" type="fixed">
-        <origin xyz="-0.1 0.0 0.0"/>
-        <parent link="base_link"/>
-        <child link="chassis_link"/>
-    </joint>
-    <!-- Chassis Link -->
-    <link name="chassis_link">
-        <visual>
-            <origin xyz="${chassis_l/2} 0 ${chassis_h/2}"/>
-            <geometry>
-                <box size="${chassis_l} ${chassis_w} ${chassis_h}"/>
-            </geometry>
-            <material name="white"/>
-        </visual>
-        <collision>
-            <origin xyz="${chassis_l/2} 0 ${chassis_h/2}"/>
-            <geometry>
-                <box size="${chassis_l} ${chassis_w} ${chassis_h}"/>
-            </geometry>
-        </collision>
-        <xacro:inertial_box mass="0.5" x="${chassis_l}" y="${chassis_w}" z="${chassis_h}">
-            <origin xyz="${chassis_l/2} 0 ${chassis_h/2}"/>
-        </xacro:inertial_box>
-    </link>
-    <!-- Left Wheel Joint -->
-    <joint name="left_wheel_joint" type="continuous">
-        <origin xyz="0.0 0.175 0.0" rpy="-${pi/2} 0.0 0.0"/>
-        <parent link="base_link"/>
-        <child link="left_wheel_link"/>
-        <axis xyz="0.0 0.0 1.0"/>
-    </joint>
-    <!-- Left Wheel Link -->
-    <link name="left_wheel_link">
-        <visual>
-            <geometry>
-                <cylinder length="${wheel_l}" radius="${wheel_r}"/>
-            </geometry>
-            <material name="blue"/>
-        </visual>
-        <collision>
-            <geometry>
-                <cylinder length="${wheel_l}" radius="${wheel_r}"/>
-            </geometry>
-        </collision>
-        <xacro:inertial_cylinder mass="0.1" length="${wheel_l}" radius="${wheel_r}">
-            <origin xyz="0 0 0" rpy="0 0 0"/>
-        </xacro:inertial_cylinder>
-    </link>
-    <!-- Right Wheel Joint -->
-    <joint name="right_wheel_joint" type="continuous">
-        <origin xyz="0.0 -0.175 0.0" rpy="${pi/2} 0.0 0.0"/>
-        <parent link="base_link"/>
-        <child link="right_wheel_link"/>
-        <axis xyz="0.0 0.0 -1.0"/>
-    </joint>
-    <!-- Right Wheel Link -->
-    <link name="right_wheel_link">
-        <visual>
-            <geometry>
-                <cylinder length="${wheel_l}" radius="${wheel_r}"/>
-            </geometry>
-            <material name="blue"/>
-        </visual>
-        <collision>
-            <geometry>
-                <cylinder length="${wheel_l}" radius="${wheel_r}"/>
-            </geometry>
-        </collision>
-        <xacro:inertial_cylinder mass="0.1" length="${wheel_l}" radius="${wheel_r}">
-            <origin xyz="0 0 0" rpy="0 0 0"/>
-        </xacro:inertial_cylinder>
-    </link>
-    <!-- Caster Wheel Joint -->
-    <joint name="caster_wheel_joint" type="fixed">
-        <origin xyz="0.24 0.0 0.0" rpy="0.0 0.0 0.0"/>
-        <parent link="chassis_link"/>
-        <child link="caster_wheel_link"/>
-        <axis xyz="0.0 0.0 -1.0"/>
-    </joint>
-    <!-- Caster Wheel Link -->
-    <link name="caster_wheel_link">
-        <visual>
-            <geometry>
-                <sphere radius="${wheel_r}"/>
-            </geometry>
-            <material name="black"/>
-        </visual>
-        <collision>
-            <geometry>
-                <sphere radius="${wheel_r}"/>
-            </geometry>
-        </collision>
-        <xacro:inertial_sphere mass="0.1" radius="${wheel_r}">
-            <origin xyz="0 0 0" rpy="0 0 0"/>
-        </xacro:inertial_sphere>
-    </link>
+    <!-- Robot Core -->
+    <xacro:include filename="dbot_mobile_core.xacro"/>
+    <!-- Gazebo -->
+    <xacro:include filename="dbot_mobile_gazebo_control.xacro"/>
 </robot>

Commit message: laser and camera

File: urdf/dbot_mobile.urdf.xacro (robot description, xacro)
@@ -7,3 +7,7 @@
     <!-- Gazebo -->
     <xacro:include filename="dbot_mobile_gazebo_control.xacro"/>
+    <!-- Lidar -->
+    <xacro:include filename="lidar.xacro"/>
+    <!-- Lidar -->
+    <xacro:include filename="camera.xacro"/>
 </robot>

File: urdf/robot_common.xacro (robot description, xacro)
@@ -9,4 +9,7 @@
     <material name="blue">
         <color rgba="0.2 0.2 1 1"/>
+    </material>
+    <material name="red">
+        <color rgba="1 0.2 0.2 1"/>
     </material>
     <material name="black">
