Commit message: working

File: urdf/dbot_mobile_core.xacro (robot description, xacro)
@@ -25,5 +25,5 @@
                 <box size="${chassis_l} ${chassis_w} ${chassis_h}"/>
             </geometry>
-            <material name="white"/>
+            <material name="orange"/>
         </visual>
         <collision>
@@ -38,5 +38,5 @@
     </link>
     <gazebo reference="chassis_link">
-        <material>Gazebo/White</material>
+        <material>Gazebo/Orange</material>
     </gazebo>
     <!-- Left Wheel Joint -->

File: urdf/dbot_mobile_gazebo_ros2_control.urdf.xacro (robot description, xacro)
@@ -6,7 +6,5 @@
     <xacro:include filename="dbot_mobile_core.xacro"/>
     <!-- Gazebo/Ros2 Control -->
-    <!-- <xacro:include filename="dbot_mobile_gazebo.xacro"/> -->
-    <!-- <xacro:include filename="dbot_mobile_gazebo_ros2_control.xacro"/> -->
-    <xacro:include filename="dbot_mobile_fake_hardware_control.xacro"/>
+    <xacro:include filename="dbot_mobile_gazebo_ros2_control.xacro"/>
     <!-- Lidar -->
     <xacro:include filename="lidar.xacro"/>

Commit message: add notes

File: urdf/dbot_mobile_core.xacro (robot description, xacro)
@@ -11,4 +11,12 @@
     <!-- Fixed base-->
     <link name="base_link">
+    </link>
+    <!-- Base Footprint Joint -->
+    <joint name="base_footprint_joint" type="fixed">
+        <origin xyz="-0.1 0.0 0.0"/>
+        <parent link="base_link"/>
+        <child link="base_footprint_link"/>
+    </joint>
+    <link name="base_footprint_link">
     </link>
     <!-- Chassis Joint -->

Commit message: update

File: urdf/dbot_mobile_core.xacro (robot description, xacro)
@@ -16,7 +16,7 @@
         <origin xyz="-0.1 0.0 0.0"/>
         <parent link="base_link"/>
-        <child link="base_footprint_link"/>
+        <child link="base_footprint"/>
     </joint>
-    <link name="base_footprint_link">
+    <link name="base_footprint">
     </link>
     <!-- Chassis Joint -->
